Commit message: Enable proper configuration

File: bundle/deepracer_simulation_environment/share/deepracer_simulation_environment/urdf/deepracer/deepracer_single_cam_lidar.urdf (robot description, URDF)
Before this commit: robot deepracer_single_cam_lidar, 12 links, 11 joints
Links:
- added link imu_link, mass 0
Joints:
- added joint car_imu_joint: type fixed, parent chassis, child imu_link, origin xyz=0 0 0 rpy=0 0 0, axis 0 0 0

File: bundle/deepracer_simulation_environment/share/deepracer_simulation_environment/urdf/deepracer/deepracer_stereo_cam.urdf (robot description, URDF)
Before this commit: robot deepracer_stereo_cam, 13 links, 12 joints
Links:
- added link imu_link, mass 0
Joints:
- added joint car_imu_joint: type fixed, parent chassis, child imu_link, origin xyz=0 0 0 rpy=0 0 0, axis 0 0 0
